File: schematic/Robot.sch (EAGLE design)
At the start: 51 parts, among them IC1 MEGA8-P, IC2 L293D, IC3 MAX232, Q1 16MHz, T1 BC337, X1 Batt, X2 Left, X3 Right, X4 RS-232

Commit message: Add files via upload
Parts:
- added JP4: Inverse, jumper:JP1E
- added R17: 4K7, rcl:R-EU_0204/7
Connections:
- new net N$1: JP4.1, R17.2
- net GND: now also R17.1
- net N$47: no longer R14.2
- net N$49: now also R14.2
- net N$53: now also JP4.2
Other:
- moved on the sheet: C7, Q1, S1
Changed lines of the file:
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@@
 <part name="SUPPLY17" library="supply2" deviceset="GND" device=""/>
 <part name="SUPPLY18" library="supply2" deviceset="+5V" device=""/>
-<part name="FRAME1" library="frames" deviceset="A3L-LOC" device=""/>
+<part name="FRAME1" library="frames2" deviceset="A3L-LOC" device=""/>
+<part name="JP4" library="jumper" deviceset="JP1E" device="" value="Inverse"/>
+<part name="R17" library="rcl" deviceset="R-EU_" device="0204/7" value="4K7"/>
+<part name="SUPPLY19" library="supply2" deviceset="GND" device=""/>
 </parts>
 <sheets>
 <sheet>
 <plain>
-<text x="194.31" y="-127" size="2.54" layer="94">Tim Dorssers</text>
-<text x="140.97" y="-132.08" size="2.54" layer="94">Line following and collision
+<text x="151.13" y="-101.6" size="2.54" layer="94">Tim Dorssers</text>
+<text x="97.79" y="-106.68" size="2.54" layer="94">Line following and collision
 avoiding robot using ATmega8</text>
 </plain>
@@
 <instance part="C5" gate="G$1" x="-91.44" y="-7.62" rot="R90"/>
 <instance part="C6" gate="G$1" x="-91.44" y="-12.7" rot="R90"/>
-<instance part="C7" gate="G$1" x="-78.74" y="-33.02"/>
+<instance part="C7" gate="G$1" x="-81.28" y="-33.02"/>
 <instance part="C8" gate="G$1" x="99.06" y="-27.94"/>
 <instance part="C9" gate="G$1" x="60.96" y="-78.74"/>
 <instance part="SUPPLY1" gate="+5V" x="-73.66" y="22.86"/>
-<instance part="SUPPLY2" gate="+5V" x="-78.74" y="-40.64" rot="R180"/>
+<instance part="SUPPLY2" gate="+5V" x="-81.28" y="-40.64" rot="R180"/>
 <instance part="SUPPLY3" gate="+5V" x="93.98" y="-22.86"/>
 <instance part="SUPPLY4" gate="+5V" x="30.48" y="55.88"/>
@@
 <instance part="SUPPLY6" gate="GND" x="60.96" y="-86.36"/>
 <instance part="SUPPLY7" gate="GND" x="157.48" y="-63.5"/>
-<instance part="Q1" gate="G$1" x="-78.74" y="-20.32" rot="R90"/>
+<instance part="Q1" gate="G$1" x="-81.28" y="-20.32" rot="R90"/>
 <instance part="C10" gate="G$1" x="-88.9" y="-22.86" rot="R270"/>
 <instance part="C11" gate="G$1" x="-88.9" y="-17.78" rot="R270"/>
 <instance part="L1" gate="G$1" x="-81.28" y="15.24"/>
-<instance part="S1" gate="1" x="-88.9" y="2.54" rot="R270"/>
+<instance part="S1" gate="1" x="-91.44" y="2.54" rot="R270"/>
 <instance part="S2" gate="1" x="-86.36" y="-73.66"/>
 <instance part="SUPPLY8" gate="GND" x="30.48" y="17.78"/>
@@
 <instance part="SUPPLY17" gate="GND" x="-43.18" y="-91.44"/>
 <instance part="SUPPLY18" gate="+5V" x="-43.18" y="-81.28"/>
-<instance part="FRAME1" gate="G$1" x="-149.86" y="-147.32"/>
+<instance part="FRAME1" gate="G$1" x="-111.76" y="-121.92"/>
+<instance part="JP4" gate="A" x="-25.4" y="-99.06" rot="R90"/>
+<instance part="R17" gate="G$1" x="-22.86" y="-104.14" rot="R90"/>
+<instance part="SUPPLY19" gate="GND" x="-22.86" y="-111.76"/>
 </instances>
 <busses>
@@
 <wire x1="-73.66" y1="10.16" x2="-73.66" y2="7.62" width="0.1524" layer="91"/>
 <wire x1="-73.66" y1="7.62" x2="-73.66" y2="0" width="0.1524" layer="91"/>
-<wire x1="-73.66" y1="0" x2="-83.82" y2="0" width="0.1524" layer="91"/>
-<wire x1="-83.82" y1="0" x2="-83.82" y2="2.54" width="0.1524" layer="91"/>
+<wire x1="-73.66" y1="0" x2="-86.36" y2="0" width="0.1524" layer="91"/>
+<wire x1="-86.36" y1="0" x2="-86.36" y2="2.54" width="0.1524" layer="91"/>
 <wire x1="-10.16" y1="-86.36" x2="-15.24" y2="-86.36" width="0.1524" layer="91"/>
 <wire x1="-15.24" y1="-86.36" x2="-15.24" y2="7.62" width="0.1524" layer="91"/>
 <wire x1="-15.24" y1="7.62" x2="-73.66" y2="7.62" width="0.1524" layer="91"/>
-<junction x="-83.82" y="0"/>
+<junction x="-86.36" y="0"/>
 <junction x="-73.66" y="0"/>
 <junction x="-73.66" y="7.62"/>
@@
 </segment>
 <segment>
-<wire x1="-78.74" y1="-38.1" x2="-73.66" y2="-38.1" width="0.1524" layer="91"/>
+<wire x1="-81.28" y1="-38.1" x2="-73.66" y2="-38.1" width="0.1524" layer="91"/>
 <wire x1="-73.66" y1="-38.1" x2="-73.66" y2="-35.56" width="0.1524" layer="91"/>
-<junction x="-78.74" y="-38.1"/>
+<junction x="-81.28" y="-38.1"/>
 <pinref part="SUPPLY2" gate="+5V" pin="+5V"/>
 <pinref part="C7" gate="G$1" pin="2"/>
@@
 </segment>
 <segment>
-<wire x1="-96.52" y1="-30.48" x2="-78.74" y2="-30.48" width="0.1524" layer="91"/>
-<wire x1="-73.66" y1="-30.48" x2="-78.74" y2="-30.48" width="0.1524" layer="91"/>
+<wire x1="-96.52" y1="-30.48" x2="-81.28" y2="-30.48" width="0.1524" layer="91"/>
+<wire x1="-73.66" y1="-30.48" x2="-81.28" y2="-30.48" width="0.1524" layer="91"/>
 <wire x1="-96.52" y1="-30.48" x2="-96.52" y2="-22.86" width="0.1524" layer="91"/>
 <wire x1="-93.98" y1="-22.86" x2="-96.52" y2="-22.86" width="0.1524" layer="91"/>
@@
 <wire x1="-73.66" y1="-5.08" x2="-96.52" y2="-5.08" width="0.1524" layer="91"/>
 <wire x1="-96.52" y1="-5.08" x2="-96.52" y2="0" width="0.1524" layer="91"/>
-<wire x1="-96.52" y1="0" x2="-93.98" y2="0" width="0.1524" layer="91"/>
-<wire x1="-93.98" y1="0" x2="-93.98" y2="2.54" width="0.1524" layer="91"/>
-<junction x="-78.74" y="-30.48"/>
-<junction x="-93.98" y="0"/>
+<wire x1="-96.52" y1="0" x2="-96.52" y2="2.54" width="0.1524" layer="91"/>
+<junction x="-81.28" y="-30.48"/>
+<junction x="-96.52" y="0"/>
 <junction x="-96.52" y="-5.08"/>
 <junction x="-96.52" y="-7.62"/>
@@
 <pinref part="S1" gate="1" pin="P"/>
 </segment>
+<segment>
+<pinref part="R17" gate="G$1" pin="1"/>
+<pinref part="SUPPLY19" gate="GND" pin="GND"/>
+</segment>
 </net>
 <net name="N$21" class="0">
 <segment>
-<wire x1="-78.74" y1="-22.86" x2="-73.66" y2="-22.86" width="0.1524" layer="91"/>
-<wire x1="-86.36" y1="-22.86" x2="-78.74" y2="-22.86" width="0.1524" layer="91"/>
-<junction x="-78.74" y="-22.86"/>
+<wire x1="-81.28" y1="-22.86" x2="-73.66" y2="-22.86" width="0.1524" layer="91"/>
+<wire x1="-86.36" y1="-22.86" x2="-81.28" y2="-22.86" width="0.1524" layer="91"/>
+<junction x="-81.28" y="-22.86"/>
 <pinref part="IC1" gate="G$1" pin="PB7(XTAL2/TOSC2)"/>
 <pinref part="Q1" gate="G$1" pin="1"/>
@@
 <net name="N$20" class="0">
 <segment>
-<wire x1="-86.36" y1="-17.78" x2="-78.74" y2="-17.78" width="0.1524" layer="91"/>
-<wire x1="-78.74" y1="-17.78" x2="-73.66" y2="-17.78" width="0.1524" layer="91"/>
-<junction x="-78.74" y="-17.78"/>
+<wire x1="-86.36" y1="-17.78" x2="-81.28" y2="-17.78" width="0.1524" layer="91"/>
+<wire x1="-81.28" y1="-17.78" x2="-73.66" y2="-17.78" width="0.1524" layer="91"/>
+<junction x="-81.28" y="-17.78"/>
 <pinref part="C11" gate="G$1" pin="1"/>
 <pinref part="IC1" gate="G$1" pin="PB6(XTAL1/TOSC1)"/>
@@
 <net name="N$47" class="0">
 <segment>
-<wire x1="20.32" y1="-53.34" x2="20.32" y2="-45.72" width="0.1524" layer="91"/>
 <wire x1="20.32" y1="-45.72" x2="-25.4" y2="-45.72" width="0.1524" layer="91"/>
 <wire x1="20.32" y1="-45.72" x2="20.32" y2="-25.4" width="0.1524" layer="91"/>
 <wire x1="20.32" y1="-25.4" x2="22.86" y2="-25.4" width="0.1524" layer="91"/>
-<junction x="20.32" y="-45.72"/>
-<pinref part="R14" gate="G$1" pin="2"/>
 <pinref part="IC1" gate="G$1" pin="PB0(ICP)"/>
 <pinref part="R16" gate="G$1" pin="1"/>
@@
 <pinref part="IC1" gate="G$1" pin="PB3(MOSI/OC2)"/>
 <pinref part="JP1" gate="A" pin="1"/>
+<pinref part="R14" gate="G$1" pin="2"/>
+<wire x1="20.32" y1="-53.34" x2="-17.78" y2="-53.34" width="0.1524" layer="91"/>
+<junction x="-17.78" y="-53.34"/>
 </segment>
 </net>
@@
 <pinref part="IC1" gate="G$1" pin="PB4(MISO)"/>
 <pinref part="JP1" gate="A" pin="9"/>
+<pinref part="JP4" gate="A" pin="2"/>
+<wire x1="-22.86" y1="-96.52" x2="-22.86" y2="-91.44" width="0.1524" layer="91"/>
+<junction x="-22.86" y="-91.44"/>
 </segment>
 </net>
@@
 </segment>
 </net>
+<net name="N$1" class="0">
+<segment>
+<pinref part="JP4" gate="A" pin="1"/>
+<pinref part="R17" gate="G$1" pin="2"/>
+</segment>
+</net>

Commit message: Add files via upload
Parts:
- removed C12: 100n, rcl:C-EU025-025X050
- removed JP4: Inverse, jumper:JP1E
- removed R16: 4K7, resistor:R-EU_0204/7
- removed R17: 4K7, rcl:R-EU_0204/7
- added LED3: Yellow, led:LED5MM
- added S4: Power, switch-misc:PVA2
- R12, R13: value 10K -> 390
- R15: value 390 -> 4K7
- S3: value Power -> Set; device switch-misc:PVA2 -> switch-omron:10-XX
Connections:
- removed net N$49: IC1.PB3(MOSI/OC2), JP1.1, R14.2
- net +5V: now also S41.O; no longer R12.1, S31.O
- net GND: now also LED3.C, S3.P, S3.P1, S42.O; no longer C12.2, R17.1, S32.O
- net N$1: now also LED3.A, R12.1; no longer JP4.1, R17.2
- net N$12: now also S42.P; no longer S32.P
- net N$24: now also S41.P; no longer S31.P
- net N$37: now also R14.1; no longer R15.1
- net N$43: now also R13.1; no longer R14.1
- net N$44: now also IC1.PB3(MOSI/OC2), JP1.1; no longer R12.2, R13.1
- net N$45: now also R15.1; no longer C12.1, R13.2
- net N$46: now also R14.2; no longer R15.2
- net N$47: now also R13.2; no longer R16.1
- net N$48: now also R15.2; no longer R16.2
- net N$52: now also S3.S, S3.S1
- net N$53: now also R12.2; no longer JP4.2
Other:
- moved on the sheet: JP1, LED1, LED2, R12, R13, R14, R15
